File: Design/uBridge1.0.sch (EAGLE design)
At the start: 45 parts, among them CN1 SATA-7, CN2 SATA-7, IC4 AP6503SP-13

Commit message: Final release of uBridge
Parts:
- removed C11: 22uF 35V 20% JB 1206, rcl:C-EUC1206
- removed C12: 100nF/S2, rcl:C-EUC0603
- removed C13: 22uf, rcl:C-EUC1206
- removed C14: 10nF/S, rcl:C-EUC0603
- removed C15: 10nF/S2, rcl:C-EUC0603
- removed C20, C21: 220nF, rcl:C-EUC0805K
- removed C22, C23: 10uF/S6 50V, rcl:C-EUC3225
- removed C24: PCE4554CT-ND, rcl:CPOL-EUUD-6,3X7,7
- removed C25, C26: 1nF, rcl:C-EUC0805K
- removed CN1, CN2: SATA-7, OfficineRobotiche:SATA-7
- removed E-M1, E-M2: (no value), pinhead:PINHD-2X2
- removed IC4: AP6503SP-13, OfficineRobotiche:AP6503SP-13'SO-8EP'
- removed JMP5, JMP6: 0R-JUMPC, jump-0r-smd:0R-JUMPC
- removed LP: Green, led:LEDCHIPLED_0805
- removed R10, R12: 10K0/S 1%, rcl:R-EU_R0603
- removed R11: 45K3/S 1%, rcl:R-EU_R0603
- removed R9: 100K0/S2 1%, rcl:R-EU_R0603
- removed U$2, U$3: A4950, allegro:A4950
- removed U$4, U$5: ACS723, allegro:ACS711
- added C3: 220nF, rcl:C-EUC0805K
- added C4, C5: 10uF/S6 50V, rcl:C-EUC3225
- added C6, C7: 1nF, rcl:C-EUC0805K
- added C8, C9: 100nF/S2, rcl:C-EUC0603
- added D1: ES1G-E2, diode:DIODE-DO214BA
- added H4: MOUNT-PAD-ROUND2.8, holes:MOUNT-PAD-ROUND2.8
- added J1, J2: 22-27-2051-05, con-molex:22-27-2051-05
- added JP2, JP3, JP4: (no value), SparkFun-Connectors:M03PTH
- added L1, L3: LED0805-YEL/S, led:LEDCHIPLED_0805
- added L4: LED0805-GRN/S, led:LEDCHIPLED_0805
- added PS1: (no value), Personale:MPT2
- added R6, R8: 3K3/S 1%, rcl:R-EU_R0603
- added R7: 6K49/S 1%, rcl:R-EU_R0603
- added U1, U3: A4950, OfficineRobotiche:A4950
- added U2, U4: ACS723, OfficineRobotiche:ACS711
- C1: value 100nF/S2 -> PCE4554CT-ND; device rcl:C-EUC0603 -> rcl:CPOL-EUUD-6,3X7,7
- C2: value 100nF/S2 -> 220nF; device rcl:C-EUC0603 -> rcl:C-EUC0805K
- JP1: value M02LOCK -> M02PTH; device SparkFun-Connectors:M02LOCK -> SparkFun-Connectors:M02PTH
- L2: value 10uH_520mA -> LED0805-GRN/S; device SparkFun-Passives:INDUCTOR1210 -> led:LEDCHIPLED_0805
- R1, R4: value 6K49/S 1% -> 1K/S 1%
- R3: value 3K3/S 1% -> 1K/S 1%
- R5: value 3K3/S 1% -> 6K49/S 1%
- SV1, SV2: device con-lstb:MA10-2 -> OfficineRobotiche:MA10-2
Connections:
- removed net AUX1: CN2.A+
- removed net AUX2: CN1.A+
- removed net N$10: JMP5-0R.2, SV1.2
- removed net N$15: C14.2, IC4.SW, L2.1
- removed net N$16: C15.1, IC4.CMP
- removed net N$17: C15.2, R12.2
- removed net N$2: R4.2, U$5.VOUT
- removed net N$23: JMP6-0R.2, SV1.1
- removed net N$4: C14.1, IC4.BST
- removed net N$5: LP.A, R2.1
- removed net N$6: IC4.EN, R9.1
- removed net N$8: C12.1, IC4.SS
- removed net N$9: IC4.FB, R10.1, R11.1
- new net N$12: L1.A, R1.2
- new net N$13: L2.A, R2.2
- new net N$18: R5.2, U2.VOUT
- new net N$29: R7.2, U4.VOUT
- new net VENC1-LD3: L3.A, R3.2
- new net VENC2-LD4: L4.A, R4.2
- net +12V: now also C1.+, C2.2, C3.2, C4.2, C5.2, D1.C, U1.VBB, U3.VBB; no longer C11.1, C20.2, C21.2, C22.2, C23.2, C24.+, IC4.IN, R9.2, U$2.VBB, U$3.VBB
- net +5V: now also U2.VCC, U4.VCC; no longer C13.1, L2.2, R11.2, R2.2, U$4.VCC, U$5.VCC
- net ANA1: now also C8.1, R5.1, R6.2; no longer C1.1, R1.1, R3.2
- net ANA2: now also C9.1, R7.1, R8.2; no longer C2.1, R4.1, R5.2
- net CHA1: now also J2-4.S; no longer E-M1.2
- net CHA2: now also J1-4.S; no longer E-M2.2
- net CHB1: now also J2-3.S; no longer E-M1.4
- net CHB2: now also J1-3.S; no longer E-M2.4
- net EN1: now also U1.VREF; no longer CN2.A-, U$2.VREF
- net EN2: now also U3.VREF; no longer CN1.A-, U$3.VREF
- net GND: now also C1.-, C2.1, C3.1, C4.1, C5.1, C6.2, C7.2, C8.2, C9.2, H4.MOUNT, J1-1.S, J2-1.S, JP2.3, JP3.3, JP4.3, L1.C, L2.C, L3.C, L4.C, PS3-1.1, R6.1, R8.1, U1.GND, U1.LSS, U1.PAD, U2.GND, U3.GND, U3.LSS, U3.PAD, U4.GND; no longer C1.2, C11.2, C12.2, C13.2, C2.2, C20.1, C21.1, C22.1, C23.1, C24.-, C25.2, C26.2, CN1.GND@1, CN1.GND@2, CN1.GND@3, CN1.H1, CN1.H2, CN2.GND@1, CN2.GND@2, CN2.GND@3, CN2.H1, CN2.H2, E-M1.1, E-M2.1, IC4.GND, IC4.PAD, JMP5-0R.3, JMP6-0R.3, LP.C, R10.2, R12.1, R3.1, R5.1, U$2.GND, U$2.LSS, U$2.PAD, U$3.GND, U$3.LSS, U$3.PAD, U$4.GND, U$5.GND
- net IO7: now also J1-2.S, SV1.2; no longer JMP5-0R.1
- net IO8: now also J2-2.S, SV1.1; no longer JMP6-0R.1
- net N$1: now also D1.A, PS3-2.1; no longer R1.2, U$4.VOUT
- net N$14: now also U1.O2, U2.IP3-, U2.IP4-; no longer U$2.O2, U$4.IP3-, U$4.IP4-
- net N$19: now also U3.O2, U4.IP3-, U4.IP4-; no longer U$3.O2, U$5.IP3-, U$5.IP4-
- net N$20: now also PS1-2.1, R2.1, U2.IP1+, U2.IP2+; no longer PS2-1.1, U$4.IP1+, U$4.IP2+
- net N$24: now also PS2-2.1, R4.1, U4.IP1+, U4.IP2+; no longer PS3-1.1, U$5.IP1+, U$5.IP2+
- net N$25: now also PS1-1.1, R1.1, U1.O1; no longer PS2-2.1, U$2.O1
- net N$26: now also PS2-1.1, R3.1, U3.O1; no longer PS3-2.1, U$3.O1
- net N$27: now also C6.1, U2./FAULT; no longer C25.1, U$4./FAULT
- net N$28: now also C7.1, U4./FAULT; no longer C26.1, U$5./FAULT
- net PWMA1: now also U1.IN2; no longer CN2.B+, U$2.IN2
- net PWMA2: now also U3.IN2; no longer CN1.B+, U$3.IN2
- net PWMB1: now also U1.IN1; no longer CN2.B-, U$2.IN1
- net PWMB2: now also U3.IN1; no longer CN1.B-, U$3.IN1
- net RX1: now also JP2.2
- net RX2: now also JP3.2
- net SCL: now also JP4.1
- net SDA: now also JP4.2
- net TX1: now also JP2.1
- net TX2: now also JP3.1
- net VENC: now also J1-5.S, J2-5.S; no longer E-M1.3, E-M2.3
Other:
- note added: "Battery"
- note added: "uNav"
- note removed: "5V Power Supply"
- note removed: "V Input : 6-23V V Output : 5V Max output current : 600mA"
